File: hardware/badge-hackgdl-2025.kicad_sch (KiCad schematic)
At the start: 53 parts, among them J1 ADDON, J2 Battery, P1 USB_C_Plug_USB2.0, Q1 DMG3415U-7, Q2 MMBT2222A, SW1 ON, SW2 RESET, SW3 BOOT, SW4 LEFT, SW5 BACK, SW6 RIGHT, SW7 MIDDLE, U1 XC6220B331MR-G, U2 ESP32-S3-WROOM-1-N16

Commit message: feat(hw): add 3d models
Parts:
- C1, C2: manf# GRM188R61E106KA73J -> (none)
- C10, C8, C9: value .1uF -> 100nF; LCSC# C478888 -> C15725; manf# 0603F104M500NT -> (none); provedor (none) -> LCSC
- C11, C12: LCSC# (none) -> C15849; provedor (none) -> LCSC
- C13, C14, C16: LCSC# (none) -> C85713; provedor (none) -> LCSC
- C15: LCSC# (none) -> C15725; provedor (none) -> LCSC
- D1: manf# MBR120LSFT1G -> (none)
- D2, D3, D4, R5: provedor (none) -> LCSC
- D5: manf# MBR120LSF -> (none)
- DS1: LCSC# (none) -> C2890596; provedor (none) -> LCSC
- J2: manf# - -> (none); provedor - -> LCSC
- R10, R11, R8, R9: LCSC# (none) -> C99198; provedor (none) -> LCSC
- R7: LCSC# (none) -> C23150; provedor (none) -> LCSC

Commit message: feat: add GPIOs shittyaddon connector
Connections:
- net GPIO1: now reaches U2.6 (IO6)
- net GPIO1: now also J1.5 (Pin_5)
- net GPIO2: now reaches U2.7 (IO7)
- net GPIO2: now also J1.6 (Pin_6)
- no-connect marks 26 -> 22
Other:
- company: (none) -> Electronic Cats
- title: (none) -> HackGDL 2025
Changed lines of the file:
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@@
 	(generator_version "8.0")
 	(paper "A4")
+	(title_block
+		(title "HackGDL 2025")
+		(date "2025-01-06")
+		(rev "1.0")
+		(company "Electronic Cats")
+		(comment 1 "Carlos Adonai")
+		(comment 2 "Andres Sabas")
+	)
 	(junction
 		(at 78.74 45.72)
@@
 	)
 	(no_connect
-		(at 191.77 39.37)
-	)
-	(no_connect
 		(at 232.41 72.39)
 	)
@@
 	)
 	(no_connect
-		(at 152.4 170.18)
-	)
-	(no_connect
 		(at 232.41 49.53)
 	)
@@
 	)
 	(no_connect
-		(at 191.77 36.83)
-	)
-	(no_connect
-		(at 139.7 170.18)
-	)
-	(no_connect
 		(at 191.77 31.75)
 	)
@@
 	(wire
 		(pts
+			(xy 187.96 39.37) (xy 191.77 39.37)
+		)
+		(stroke
+			(width 0)
+			(type default)
+		)
+	)
+	(wire
+		(pts
 			(xy 73.66 162.56) (xy 73.66 165.1)
 		)
@@
 	(wire
 		(pts
+			(xy 152.4 170.18) (xy 154.94 170.18)
+		)
+		(stroke
+			(width 0)
+			(type default)
+		)
+	)
+	(wire
+		(pts
 			(xy 213.36 99.06) (xy 212.09 99.06)
 		)
@@
 	(wire
 		(pts
+			(xy 137.16 170.18) (xy 139.7 170.18)
+		)
+		(stroke
+			(width 0)
+			(type default)
+		)
+	)
+	(wire
+		(pts
 			(xy 54.61 154.94) (xy 57.15 154.94)
 		)
@@
 	(wire
 		(pts
+			(xy 187.96 36.83) (xy 191.77 36.83)
+		)
+		(stroke
+			(width 0)
+			(type default)
+		)
+	)
+	(wire
+		(pts
 			(xy 73.66 132.08) (xy 73.66 137.16)
 		)
@@
 	(wire
 		(pts
+			(xy 154.94 167.64) (xy 152.4 167.64)
+		)
+		(stroke
+			(width 0)
+			(type default)
+		)
+	)
+	(wire
+		(pts
 			(xy 171.45 44.45) (xy 171.45 45.593)
 		)
@@
 		(pts
 			(xy 242.57 116.84) (xy 242.57 109.22)
+		)
+		(stroke
+			(width 0)
+			(type default)
+		)
+	)
+	(wire
+		(pts
+			(xy 137.16 167.64) (xy 139.7 167.64)
 		)
 		(stroke
@@
 		)
 	)
+	(label "GPIO1"
+		(at 154.94 170.18 0)
+		(fields_autoplaced yes)
+		(effects
+			(font
+				(size 1.27 1.27)
+			)
+			(justify left bottom)
+		)
+	)
 	(label "NEOPIXEL"
 		(at 182.88 148.59 0)
@@
 	)
 	(label "SCL"
-		(at 139.7 167.64 180)
+		(at 137.16 167.64 180)
 		(fields_autoplaced yes)
 		(effects
@@
 		)
 	)
+	(label "GPIO1"
+		(at 187.96 36.83 180)
+		(fields_autoplaced yes)
+		(effects
+			(font
+				(size 1.27 1.27)
+			)
+			(justify right bottom)
+		)
+	)
 	(label "Buzz"
 		(at 158.242 120.65 0)
@@
 		)
 	)
+	(label "GPIO2"
+		(at 187.96 39.37 180)
+		(fields_autoplaced yes)
+		(effects
+			(font
+				(size 1.27 1.27)
+			)
+			(justify right bottom)
+		)
+	)
+	(label "GPIO2"
+		(at 137.16 170.18 180)
+		(fields_autoplaced yes)
+		(effects
+			(font
+				(size 1.27 1.27)
+			)
+			(justify right bottom)
+		)
+	)
 	(label "SDA"
-		(at 152.4 167.64 0)
-		(fields_autoplaced yes)
-		(effects
+		(at 154.94 167.64 0)
+		(fields_autoplaced yes)
+		(effects

Commit message: feat(hw): update bom
Parts:
- BZ1: provedor DigiKey -> MOUSER
- J1: LCSC# (none) -> C3975148; manf# M20-7810345 -> (none); provedor (none) -> LCSC
- R1, R2: LCSC# C191782 -> C309655
- R4: value 10K -> 10k
- U2: manf# (none) -> 356-ESP32-S3WROOM1N4
Changed lines of the file:
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@@
 			)
 		)
-		(property "LCSC#" "C191782"
+		(property "LCSC#" "C309655"
 			(at 50.8 34.29 0)
 			(effects
@@
 			)
 		)
-		(property "Value" "10K"
+		(property "Value" "10k"
 			(at 176.276 40.132 0)
 			(effects
@@
 			)
 		)
+		(property "manf#" "356-ESP32-S3WROOM1N4"
+			(at 191.77 24.13 0)
+			(effects
+				(font
+					(size 1.27 1.27)
+				)
+				(hide yes)
+			)
+		)
 		(pin "1"
 		)
@@
 			)
 		)
-		(property "LCSC#" ""
+		(property "LCSC#" "C3975148"
 			(at 147.32 167.64 0)
 			(effects
@@
 			)
 		)
-		(property "manf#" "M20-7810345 "
+		(property "manf#" ""
+			(at 147.32 167.64 0)
+			(effects
+				(font
+					(size 1.27 1.27)
+				)
+				(hide yes)
+			)
+		)
+		(property "provedor" "LCSC"
 			(at 147.32 167.64 0)
 			(effects
@@
 			)
 		)
-		(property "provedor" "DigiKey"
+		(property "provedor" "MOUSER"
 			(at 130.81 110.49 0)
 			(effects
@@
 			)
 		)
-		(property "LCSC#" "C191782"
+		(property "LCSC#" "C309655"
 			(at 50.8 31.75 0)
 			(effects
